Commit message: CHỈNH SỬA MODEL, THÊM WORLDS
- Chỉnh sửa laser scan một chút để hiển thị vùng quét
- Thêm obstacle world

File: urdf/sensor_wheel_robot.xacro (robot description, xacro)
@@ -1,175 +1,168 @@
-<?xml version="1.0"?>
-<robot  xmlns:xacro="http://www.ros.org/wiki/xacro"
-	xmlns:sensor="http://playerstage.sourceforge.net/gazebo/xmlschema/#sensor"
-    	xmlns:controller="http://playerstage.sourceforge.net/gazebo/xmlschema/#controller"
-    	xmlns:interface="http://playerstage.sourceforge.net/gazebo/xmlschema/#interface"
-	name="wheel_robot_xacro">
- 	<!-- Parameters declaration -->
-	<xacro:property name="length_wheel" value="0.05" />
-	<xacro:property name="radius_wheel" value="0.05" />
-	<xacro:property name="camera_link" value="0.05" />
-	<xacro:property name="hokuyo_size" value="0.05" />
-	<xacro:macro name="default_inertial" params="mass">
-               <inertial>
-                       <mass value="${mass}" />
-                       <inertia ixx="1.0" ixy="0.0" ixz="0.0"
-                                iyy="1.0" iyz="0.0"
-                                izz="1.0" />
-               </inertial>
-	</xacro:macro>
-	<xacro:include filename="$(find robot_gazebo)/urdf/robot.gazebo" />
-	<link name="base_footprint">
-   		<visual>
-			<geometry>
-      				<box size="0.001 0.001 0.001"/>
-     			</geometry>
-			<origin rpy="0 0 0" xyz="0 0 0"/>
-   		</visual>
-		<xacro:default_inertial mass="0.0001"/>
- 	</link>
-	<gazebo reference="base_footprint">
-		<material>Gazebo/Green</material>
-		<turnGravityOff>false</turnGravityOff>
-	</gazebo>
-	<joint name="base_footprint_joint" type="fixed">
-		<origin xyz="0 0 0" />
-		<parent link="base_footprint" />
-		<child link="base_link" />
-	</joint>
-	<link name="base_link">
-   		<visual>
-			<geometry>
-      				<box size="0.2 .3 .1"/>
-     			</geometry>
-			<origin rpy="0 0 1.54" xyz="0 0 0.05"/>
-			<material name="white">
-				<color rgba="1 1 1 1"/>
-			</material>
-   		</visual>
-		<collision>
-			<geometry>
-       				<box size="0.2 .3 0.1"/>
-			</geometry>
-		</collision>
-		<xacro:default_inertial mass="10"/>
- 	</link>
- 	<link name="wheel_1">
-   		<visual>
-     			<geometry>
-       				<cylinder length="${length_wheel}" radius="${radius_wheel}"/>
-     			</geometry>
-			<!-- <origin rpy="0 1.5 0" xyz="0.1 0.1 0"/> -->
-			<origin rpy="0 0 0" xyz="0 0 0"/>
-   			<material name="black">
-				<color rgba="0 0 0 1"/>
-			</material>
-		</visual>
-		<collision>
-			<geometry>
-       				<cylinder length="${length_wheel}" radius="${radius_wheel}"/>
-			</geometry>
-		</collision>
-		<xacro:default_inertial mass="1"/>
- 	</link>
- 	<link name="wheel_2">
-   		<visual>
-     			<geometry>
-       				<cylinder length="${length_wheel}" radius="${radius_wheel}"/>
-     			</geometry>
-			<!-- <origin rpy="0 1.5 0" xyz="-0.1 0.1 0"/> -->
-			<origin rpy="0 0 0" xyz="0 0 0"/>
-   			<material name="black"/>
-   		</visual>
-		<collision>
-			<geometry>
-       				<cylinder length="${length_wheel}" radius="${radius_wheel}"/>
-			</geometry>
-		</collision>
-		<xacro:default_inertial mass="1"/>
- 	</link>
- 	<link name="wheel_3">
-   		<visual>
-     			<geometry>
-       				<cylinder length="${length_wheel}" radius="${radius_wheel}"/>
-     			</geometry>
-			<!-- <origin rpy="0 1.5 0" xyz="0.1 -0.1 0"/> -->
-			<origin rpy="0 0 0" xyz="0 0 0"/>
-   			<material name="black"/>
-   		</visual>
-		<collision>
-			<geometry>
-       				<cylinder length="${length_wheel}" radius="${radius_wheel}"/>
-			</geometry>
-		</collision>
-		<xacro:default_inertial mass="1"/>
- 	</link>
- 	<link name="wheel_4">
-   		<visual>
-     			<geometry>
-       				<cylinder length="${length_wheel}" radius="${radius_wheel}"/>
-     			</geometry>
-		<!--	<origin rpy="0 1.5 0" xyz="-0.1 -0.1 0"/> -->
-			<origin rpy="0 0 0" xyz="0 0 0" />
-   			<material name="black"/>
-   		</visual>
-		<collision>
-			<geometry>
-       				<cylinder length="${length_wheel}" radius="${radius_wheel}"/>
-			</geometry>
-		</collision>
-		<xacro:default_inertial mass="1"/>
- 	</link>
-	<!-- Adding Hokuyo Laser -->
-  	<link name="hokuyo_link">
-    		<collision>
-    			<origin xyz="0 0 0" rpy="0 0 0"/>
-      			<geometry>
-				<box size="0.1 0.1 0.1"/>
-      			</geometry>
-    		</collision>
-   		<visual>
-      			<origin xyz="0 0 0" rpy="0 0 0"/>
-      			<geometry>
-        			<mesh filename="package://robot_gazebo/meshes/hokuyo.dae"/>
-      			</geometry>
-    		</visual>
-    		<inertial>
-      			<mass value="1e-5" />
-      			<origin xyz="0 0 0" rpy="0 0 0"/>
-      			<inertia ixx="1e-6" ixy="0" ixz="0" iyy="1e-6" iyz="0" izz="1e-6" />
-    		</inertial>
-  	</link>
-		<!-- Joint declartion -->
- 	<joint name="base_to_wheel1" type="continuous">
-  		 <parent link="base_link"/>
- 		 <child link="wheel_1"/>
-  		 <origin rpy="1.5707 0 0" xyz="0.1 0.15 0"/>
-   		 <axis xyz="0 0 1" />
- 	</joint>
- 	<joint name="base_to_wheel2" type="continuous">
- 	 	<axis xyz="0 0 1" />
-   		<anchor xyz="0 0 0" />
-  		<limit effort="100" velocity="100" />
-   		<parent link="base_link"/>
-   		<child link="wheel_2"/>
-   		<origin rpy="1.5707 0 0" xyz="-0.1 0.15 0"/>
-	</joint>
-	<joint name="base_to_wheel3" type="continuous">
-   		<parent link="base_link"/>
-   		<axis xyz="0 0 1" />
-   		<child link="wheel_3"/>
-   		<origin rpy="1.5707 0 0" xyz="0.1 -0.15 0"/>
- 	</joint>
- 	<joint name="base_to_wheel4" type="continuous">
-   		<parent link="base_link"/>
-   		<axis xyz="0 0 1" />
-   		<child link="wheel_4"/>
-   		<origin rpy="1.5707 0 0" xyz="-0.1 -0.15 0"/>
- 	</joint>
-	<joint name="hokuyo_joint" type="fixed">
-    		<axis xyz="0 1 0" />
-    		<origin xyz="0.125 0.05 0.125" rpy="0 0 0"/>
-    		<parent link="base_link"/>
-    		<child link="hokuyo_link"/>
-  	</joint>
+<?xml version="1.0" encoding="UTF-8"?>
+<robot  xmlns:xacro="http://www.ros.org/wiki/xacro" 	xmlns:sensor="http://playerstage.sourceforge.net/gazebo/xmlschema/#sensor"    	xmlns:controller="http://playerstage.sourceforge.net/gazebo/xmlschema/#controller"    	xmlns:interface="http://playerstage.sourceforge.net/gazebo/xmlschema/#interface"	name="wheel_robot_xacro">
+  <!-- Parameters declaration -->
+  <xacro:property name="length_wheel" value="0.05" />
+  <xacro:property name="radius_wheel" value="0.05" />
+  <xacro:property name="camera_link" value="0.05" />
+  <xacro:property name="hokuyo_size" value="0.05" />
+  <xacro:macro name="default_inertial" params="mass">
+    <inertial>
+      <mass value="${mass}" />
+      <inertia ixx="1.0" ixy="0.0" ixz="0.0"                                iyy="1.0" iyz="0.0"                                izz="1.0" />
+    </inertial>
+  </xacro:macro>
+  <xacro:include filename="$(find robot_gazebo)/urdf/robot.gazebo" />
+  <link name="base_footprint">
+    <visual>
+      <geometry>
+        <box size="0.001 0.001 0.001"/>
+      </geometry>
+      <origin rpy="0 0 0" xyz="0 0 0"/>
+    </visual>
+    <xacro:default_inertial mass="0.0001"/>
+  </link>
+  <gazebo reference="base_footprint">
+    <material>Gazebo/Green</material>
+    <turnGravityOff>false</turnGravityOff>
+  </gazebo>
+  <joint name="base_footprint_joint" type="fixed">
+    <origin xyz="0 0 0" />
+    <parent link="base_footprint" />
+    <child link="base_link" />
+  </joint>
+  <link name="base_link">
+    <visual>
+      <geometry>
+        <box size="0.2 .3 .1"/>
+      </geometry>
+      <origin rpy="0 0 1.54" xyz="0 0 0.05"/>
+      <material name="white">
+        <color rgba="1 1 1 1"/>
+      </material>
+    </visual>
+    <collision>
+      <geometry>
+        <box size="0.2 .3 0.1"/>
+      </geometry>
+    </collision>
+    <xacro:default_inertial mass="10"/>
+  </link>
+  <link name="wheel_1">
+    <visual>
+      <geometry>
+        <cylinder length="${length_wheel}" radius="${radius_wheel}"/>
+      </geometry>
+      <!-- <origin rpy="0 1.5 0" xyz="0.1 0.1 0"/> -->
+      <origin rpy="0 0 0" xyz="0 0 0"/>
+      <material name="black">
+        <color rgba="0 0 0 1"/>
+      </material>
+    </visual>
+    <collision>
+      <geometry>
+        <cylinder length="${length_wheel}" radius="${radius_wheel}"/>
+      </geometry>
+    </collision>
+    <xacro:default_inertial mass="1"/>
+  </link>
+  <link name="wheel_2">
+    <visual>
+      <geometry>
+        <cylinder length="${length_wheel}" radius="${radius_wheel}"/>
+      </geometry>
+      <!-- <origin rpy="0 1.5 0" xyz="-0.1 0.1 0"/> -->
+      <origin rpy="0 0 0" xyz="0 0 0"/>
+      <material name="black"/>
+    </visual>
+    <collision>
+      <geometry>
+        <cylinder length="${length_wheel}" radius="${radius_wheel}"/>
+      </geometry>
+    </collision>
+    <xacro:default_inertial mass="1"/>
+  </link>DA  <link name="wheel_3">
+  <visual>
+    <geometry>
+      <cylinder length="${length_wheel}" radius="${radius_wheel}"/>
+    </geometry>
+    <!-- <origin rpy="0 1.5 0" xyz="0.1 -0.1 0"/> -->
+    <origin rpy="0 0 0" xyz="0 0 0"/>
+    <material name="black"/>
+  </visual>
+  <collision>
+    <geometry>
+      <cylinder length="${length_wheel}" radius="${radius_wheel}"/>
+    </geometry>
+  </collision>
+  <xacro:default_inertial mass="1"/>
+</link>
+<link name="wheel_4">
+  <visual>
+    <geometry>
+      <cylinder length="${length_wheel}" radius="${radius_wheel}"/>
+    </geometry>
+    <!--	<origin rpy="0 1.5 0" xyz="-0.1 -0.1 0"/> -->
+    <origin rpy="0 0 0" xyz="0 0 0" />
+    <material name="black"/>
+  </visual>
+  <collision>
+    <geometry>
+      <cylinder length="${length_wheel}" radius="${radius_wheel}"/>
+    </geometry>
+  </collision>
+  <xacro:default_inertial mass="1"/>
+</link>
+<!-- Adding Hokuyo Laser -->
+<link name="hokuyo_link">
+  <collision>
+    <origin xyz="0 0 0" rpy="0 0 0"/>
+    <geometry>
+      <box size="0.1 0.1 0.1"/>
+    </geometry>
+  </collision>
+  <visual>
+    <origin xyz="0 0 0" rpy="0 0 0"/>
+    <geometry>
+      <mesh filename="package://robot_gazebo/meshes/hokuyo.dae"/>
+    </geometry>
+  </visual>
+  <inertial>
+    <mass value="1e-5" />
+    <origin xyz="0 0 0" rpy="0 0 0"/>
+    <inertia ixx="1e-6" ixy="0" ixz="0" iyy="1e-6" iyz="0" izz="1e-6" />
+  </inertial>
+</link>
+<!-- Joint declartion -->
+<joint name="base_to_wheel1" type="continuous">
+  <parent link="base_link"/>
+  <child link="wheel_1"/>
+  <origin rpy="1.5707 0 0" xyz="0.1 0.15 0"/>
+  <axis xyz="0 0 1" />
+</joint>
+<joint name="base_to_wheel2" type="continuous">
+  <axis xyz="0 0 1" />
+  <anchor xyz="0 0 0" />
+  <limit effort="100" velocity="100" />
+  <parent link="base_link"/>
+  <child link="wheel_2"/>
+  <origin rpy="1.5707 0 0" xyz="-0.1 0.15 0"/>
+</joint>
+<joint name="base_to_wheel3" type="continuous">
+  <parent link="base_link"/>
+  <axis xyz="0 0 1" />
+  <child link="wheel_3"/>
+  <origin rpy="1.5707 0 0" xyz="0.1 -0.15 0"/>
+</joint>
+<joint name="base_to_wheel4" type="continuous">
+  <parent link="base_link"/>
+  <axis xyz="0 0 1" />
+  <child link="wheel_4"/>
+  <origin rpy="1.5707 0 0" xyz="-0.1 -0.15 0"/>
+</joint>
+<joint name="hokuyo_joint" type="fixed">
+  <axis xyz="0 1 0" />
+  <origin xyz="0.125 0.05 0.125" rpy="0 0 0"/>
+  <parent link="base_link"/>
+  <child link="hokuyo_link"/>
+</joint>
 </robot>
